File: PCBs/F1Wheel-UpperBlinkBoard/F1Wheel-UpperBlinkBoard.kicad_pcb (KiCad board)
At the start: 2 copper layers, 227.4 x 69.9 mm, 45 parts, among them J1 HLW20R-2C7LF, M3 MountingHole_3.2mm_M3_DIN965_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, SW1 SKQEACA010, SW2 SKQEACA010, SW3 SKQEACA010, SW4 SKQEACA010, SW5 SKQEACA010, SW6 SKQEACA010, SW7 SKQEACA010, SW8 SKQEACA010

Commit message: organization changes
Parts:
- renumbered REF** to M3
Connections:
- D13 pad 3: unconnected-(D13-GND-Pad3) -> GND
