File: PCBs/F1Wheel-UpperBlinkBoard/F1Wheel-UpperBlinkBoard.kicad_sch (KiCad schematic)
At the start: 38 parts, among them J1 HLW20R-2C7LF, SW1 SKQEACA010, SW2 SKQEACA010, SW3 SKQEACA010, SW4 SKQEACA010, SW5 SKQEACA010, SW6 SKQEACA010, SW7 SKQEACA010, SW8 SKQEACA010

Commit message: organization changes
Connections:
- net GND: now also D13.3 (GND)
Changed lines of the file:
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@@
 	(wire
 		(pts
+			(xy 274.32 25.4) (xy 270.51 25.4)
+		)
+		(stroke
+			(width 0)
+			(type default)
+		)
+	)
+	(wire
+		(pts
 			(xy 158.75 22.86) (xy 158.75 25.4)
 		)
@@
 					(unit 1)
 				)
+			)
+		)
+	)
+	(symbol
+		(lib_id "power:GND")
+		(at 274.32 25.4 0)
+		(unit 1)
+		(exclude_from_sim no)
+		(in_bom yes)
+		(on_board yes)
+		(dnp no)
+		(property "Reference" "#PWR049"
+			(at 274.32 31.75 0)
+			(effects
+				(font
+					(size 1.27 1.27)
+				)
+				(hide yes)
+			)
+		)
+		(property "Value" "GND"
+			(at 274.32 29.21 0)
+			(effects
+				(font
+					(size 1.27 1.27)
+				)
+			)
+		)
+		(property "Footprint" ""
+			(at 274.32 25.4 0)
+			(effects
+				(font
+					(size 1.27 1.27)
+				)
+				(hide yes)
+			)
+		)
+		(property "Datasheet" ""
+			(at 274.32 25.4 0)
+			(effects
+				(font
+					(size 1.27 1.27)
+				)
+				(hide yes)
+			)
+		)
+		(property "Description" "Power symbol creates a global label with name \"GND\" , ground"
+			(at 274.32 25.4 0)
+			(effects
+				(font
+					(size 1.27 1.27)
+				)
+				(hide yes)
+			)
+		)
+		(pin "1"
+		)
+		(instances
+			(project "F1Wheel-UpperBlinkBoard"
+				(path "/a6f92ccc-f41a-40f6-978a-4e53e6ac144b"
+					(reference "#PWR049")
+					(unit 1)
+				)
